File: kicad_source/vidorcameraadapter.sch (KiCad schematic (older format))
At the start: 59 parts, among them CN1 CONN_02X26, CN2 CONN_02X10, CN3 CONN_01X03

Commit message: placed all new parts in layout
Parts:
- removed D6: LED_RABG, symbol devices:LED_RABG
- added D6: LED_RGB, LEDs:LED_RGB_PLLC-6, symbol devices:LED_RGB
- D1, D2, D3, D4, D5: footprint (none) -> LEDs:LED_0603
Connections:
- wire segments 159 -> 163
Changed lines of the file:
@@
 F 0 "D5" H 8500 5995 50  0000 C CNN
 F 1 "Led_Small" H 8500 6086 50  0000 C CNN
-F 2 "" V 8500 6200 50  0000 C CNN
+F 2 "LEDs:LED_0603" V 8500 6200 50  0001 C CNN
 F 3 "" V 8500 6200 50  0000 C CNN
 	1    8500 6200
@@
 F 0 "D4" H 8500 5445 50  0000 C CNN
 F 1 "Led_Small" H 8500 5536 50  0000 C CNN
-F 2 "" V 8500 5650 50  0000 C CNN
+F 2 "LEDs:LED_0603" V 8500 5650 50  0001 C CNN
 F 3 "" V 8500 5650 50  0000 C CNN
 	1    8500 5650
@@
 F 0 "D3" H 8500 4895 50  0000 C CNN
 F 1 "Led_Small" H 8500 4986 50  0000 C CNN
-F 2 "" V 8500 5100 50  0000 C CNN
+F 2 "LEDs:LED_0603" V 8500 5100 50  0001 C CNN
 F 3 "" V 8500 5100 50  0000 C CNN
 	1    8500 5100
@@
 F 0 "D2" H 8500 4345 50  0000 C CNN
 F 1 "Led_Small" H 8500 4436 50  0000 C CNN
-F 2 "" V 8500 4550 50  0000 C CNN
+F 2 "LEDs:LED_0603" V 8500 4550 50  0001 C CNN
 F 3 "" V 8500 4550 50  0000 C CNN
 	1    8500 4550
@@
 F 0 "D1" H 8500 3795 50  0000 C CNN
 F 1 "Led_Small" H 8500 3886 50  0000 C CNN
-F 2 "" V 8500 4000 50  0000 C CNN
+F 2 "LEDs:LED_0603" V 8500 4000 50  0001 C CNN
 F 3 "" V 8500 4000 50  0000 C CNN
 	1    8500 4000
@@
 	7900 4000 7700 4000
 $Comp
-L devices:LED_RABG D6
-U 1 1 5E3EF9EF
-P 10500 5750
-F 0 "D6" H 10500 6215 50  0000 C CNN
-F 1 "LED_RABG" H 10500 6124 50  0000 C CNN
-F 2 "" H 10450 5700 50  0000 C CNN
-F 3 "" H 10450 5700 50  0000 C CNN
-	1    10500 5750
-	1    0    0    -1
-$EndComp
-$Comp
 L devices:R_0603 R32
 U 1 1 5E3F2B43
@@
 L power-supply:+3V3 #PWR012
 U 1 1 5E3F36D6
-P 10950 5650
-F 0 "#PWR012" H 10950 5500 50  0001 C CNN
-F 1 "+3V3" H 10965 5823 50  0000 C CNN
-F 2 "" H 10950 5650 50  0000 C CNN
-F 3 "" H 10950 5650 50  0000 C CNN
-	1    10950 5650
+P 10750 5500
+F 0 "#PWR012" H 10750 5350 50  0001 C CNN
+F 1 "+3V3" H 10765 5673 50  0000 C CNN
+F 2 "" H 10750 5500 50  0000 C CNN
+F 3 "" H 10750 5500 50  0000 C CNN
+	1    10750 5500
 	1    0    0    -1
 $EndComp
@@
 Wire Wire Line
 	10050 5550 10200 5550
-Wire Wire Line
-	10800 5750 10950 5750
-Wire Wire Line
-	10950 5750 10950 5650
 Text Label 9100 5550 0    50   ~ 0
 LED_R
@@
 Wire Wire Line
 	2450 4800 3300 4800
+$Comp
+L devices:LED_RGB D6
+U 1 1 5E34D3F1
+P 10400 5750
+F 0 "D6" H 10400 6215 50  0000 C CNN
+F 1 "LED_RGB" H 10400 6124 50  0000 C CNN
+F 2 "LEDs:LED_RGB_PLLC-6" H 10400 6123 50  0001 C CNN
+F 3 "" H 10400 5700 50  0000 C CNN
+	1    10400 5750
+	1    0    0    -1
+$EndComp
+Wire Wire Line
+	10600 5950 10750 5950
+Wire Wire Line
+	10750 5950 10750 5750
+Wire Wire Line
+	10600 5550 10750 5550
+Connection ~ 10750 5550
+Wire Wire Line
+	10750 5550 10750 5500
+Wire Wire Line
+	10600 5750 10750 5750
+Connection ~ 10750 5750
+Wire Wire Line
+	10750 5750 10750 5550
 $EndSCHEMATC
