File: kicad_source/vidorcameraadapter.sch (KiCad schematic (older format))
At the start: 59 parts, among them CN1 CONN_02X26, CN2 CONN_02X10, CN3 CONN_01X03

Commit message: added logo and description on silkscreen
Other:
- note added: "for use with Arducam OV2640 breakout board with M12 lens\nhttps://www.arducam.com/product/2mp-ov2640-camera-module/"
Changed lines of the file:
@@
 Wire Wire Line
 	10750 5750 10750 5550
+Text Notes 5650 1100 0    50   ~ 0
+for use with Arducam OV2640 breakout board with M12 lens\nhttps://www.arducam.com/product/2mp-ov2640-camera-module/
 $EndSCHEMATC

Commit message: added jumper for I2C pullup, added buffer ic for I2C leds, made mounting holes as parts, made DRC, updated images
Parts:
- added C1, C2: 100nF, capacitors:C_0603, symbol devices:C_0603
- added JP1, JP2: Jumper_NC_Small, wire_pads:SolderJumper_2mm, symbol devices:Jumper_NC_Small
- added MECH7, MECH8, MECH9: MHP_3.2_5.8, MECH_mounting_holes:MHP_3.2_5.8, symbol MECH_mounting-holes:MHP_3.2_5.8
- added U1: SN74LVC2G34DBV, SOT_TO:SOT-23-6, symbol IC_logic:SN74LVC2G34
- CN1: value CONN_02X26 -> TE_2041119-2
- CN2: value CONN_02X10 -> RS2-20-G
- CN3: value CONN_01X03 -> DNI
- D1: value Led_Small -> Led yellow
- D2, D4: value Led_Small -> Led green
- D3, D5: value Led_Small -> Led red
- D6: value LED_RGB -> 150353M153300
Connections:
- net labels added: SCL_B, SDA_B
- wire segments 163 -> 176
- no-connect marks 6 -> 9
Other:
- note added: "Pin 30 and 32 have \npull up on Vidor 4000"
- note added: "mounting holes"
- note removed: "Pin 30 and 32 have pull up on Vidor 4000"
- moved on the sheet: CN3, R21, R22

Commit message: moved pins on the Vidor connector to free NINA pins and pins with pull up, exchanged PCLK and XCLK, added pdfs and generated images
Other:
- note added: "Pin 1, 3, 5, 7, 17 and 19 \nare also connected to \nthe WiFi NINA module \non the Vidor 4000"
- moved on the sheet: R23, R24, W10, W11, W12, W5
Changed lines of the file:
@@
 encoding utf-8
 Sheet 1 1
-Title ""
-Date ""
-Rev ""
-Comp ""
+Title "VidorCameraAdapter"
+Date "2020-02-05"
+Rev "0.1"
+Comp "107-systems"
 Comment1 ""
 Comment2 ""
@@
 VSYNC
 Text Label 2550 5300 0    50   ~ 0
-PCLK
-Text Label 4200 5600 0    50   ~ 0
+XCLK
+Text Label 4200 4800 0    50   ~ 0
 RST
 Text Label 2550 6700 0    50   ~ 0
@@
 HREF
 Text Label 2550 5400 0    50   ~ 0
-XCLK
-Text Label 4200 5700 0    50   ~ 0
+PCLK
+Text Label 4200 4900 0    50   ~ 0
 PWDN
 Text Label 2550 6600 0    50   ~ 0
@@
 PEX_RST
 Wire Wire Line
-	4750 5700 3800 5700
-Wire Wire Line
-	4750 5600 3800 5600
+	4750 4900 3800 4900
+Wire Wire Line
+	4750 4800 3800 4800
 Text Notes 4850 5750 0    50   ~ 0
 Pin 30 and 32 have \npull up on Vidor 4000
@@
 	2650 4500 3300 4500
 Wire Wire Line
-	2650 4700 3300 4700
-Wire Wire Line
-	4500 4700 3800 4700
-Wire Wire Line
-	4500 4600 3800 4600
-Wire Wire Line
-	4500 4500 3800 4500
+	2650 5100 3300 5100
+Wire Wire Line
+	4500 5700 3800 5700
+Wire Wire Line
+	4500 5600 3800 5600
 Wire Wire Line
 	4500 4400 3800 4400
@@
 Text Label 2750 4500 0    50   ~ 0
 RSVD4
+Text Label 2750 5000 0    50   ~ 0
+RSVD5
+Text Label 4100 5600 0    50   ~ 0
+RSVD6
+Text Label 2750 5100 0    50   ~ 0
+RSVD7
+Text Label 4100 5700 0    50   ~ 0
+RSVD8
 Text Label 4100 4500 0    50   ~ 0
-RSVD5
+LED_R
 Text Label 4100 4600 0    50   ~ 0
-RSVD6
-Text Label 2750 4700 0    50   ~ 0
-RSVD7
+SDA_V
 Text Label 4100 4700 0    50   ~ 0
-RSVD8
+SCL_V
+Text Label 2550 4700 0    50   ~ 0
+LED_G
 Text Label 2550 4800 0    50   ~ 0
-LED_R
-Text Label 4100 4800 0    50   ~ 0
-SDA_V
-Text Label 4100 4900 0    50   ~ 0
-SCL_V
-Text Label 2550 5000 0    50   ~ 0
-LED_G
-Text Label 2550 5100 0    50   ~ 0
 LED_B
 $Comp
@@
 L mechanical-connectors:TEST_1P W10
 U 1 1 5E3153CE
-P 4500 4500
-F 0 "W10" V 4454 4688 50  0000 L CNN
-F 1 "TEST_1P" V 4545 4688 50  0001 L CNN
-F 2 "wire_pads:SolderWirePad_single_1mmSMD" V 4591 4688 50  0001 L CNN
-F 3 "" H 4700 4500 50  0000 C CNN
-	1    4500 4500
-	0    1    1    0
+P 2650 5000
+F 0 "W10" V 2650 5200 50  0000 L CNN
+F 1 "TEST_1P" V 2695 5188 50  0001 L CNN
+F 2 "wire_pads:SolderWirePad_single_1mmSMD" V 2741 5188 50  0001 L CNN
+F 3 "" H 2850 5000 50  0000 C CNN
+	1    2650 5000
+	0    -1   -1   0
 $EndComp
 $Comp
 L mechanical-connectors:TEST_1P W11
 U 1 1 5E31571A
-P 4500 4600
-F 0 "W11" V 4454 4788 50  0000 L CNN
-F 1 "TEST_1P" V 4545 4788 50  0001 L CNN
-F 2 "wire_pads:SolderWirePad_single_1mmSMD" V 4591 4788 50  0001 L CNN
-F 3 "" H 4700 4600 50  0000 C CNN
-	1    4500 4600
+P 4500 5600
+F 0 "W11" V 4454 5788 50  0000 L CNN
+F 1 "TEST_1P" V 4545 5788 50  0001 L CNN
+F 2 "wire_pads:SolderWirePad_single_1mmSMD" V 4591 5788 50  0001 L CNN
+F 3 "" H 4700 5600 50  0000 C CNN
+	1    4500 5600
 	0    1    1    0
 $EndComp
@@
 L mechanical-connectors:TEST_1P W12
 U 1 1 5E3158F5
-P 4500 4700
-F 0 "W12" V 4454 4888 50  0000 L CNN
-F 1 "TEST_1P" V 4545 4888 50  0001 L CNN
-F 2 "wire_pads:SolderWirePad_single_1mmSMD" V 4591 4888 50  0001 L CNN
-F 3 "" H 4700 4700 50  0000 C CNN
-	1    4500 4700
+P 4500 5700
+F 0 "W12" V 4454 5888 50  0000 L CNN
+F 1 "TEST_1P" V 4545 5888 50  0001 L CNN
+F 2 "wire_pads:SolderWirePad_single_1mmSMD" V 4591 5888 50  0001 L CNN
+F 3 "" H 4700 5700 50  0000 C CNN
+	1    4500 5700
 	0    1    1    0
 $EndComp
@@
 L mechanical-connectors:TEST_1P W5
 U 1 1 5E31885D
-P 2650 4700
-F 0 "W5" V 2650 4950 50  0000 C CNN
-F 1 "TEST_1P" V 2754 4772 50  0001 C CNN
-F 2 "wire_pads:SolderWirePad_single_1mmSMD" V 2741 4888 50  0001 L CNN
-F 3 "" H 2850 4700 50  0000 C CNN
-	1    2650 4700
+P 2650 5100
+F 0 "W5" V 2650 5350 50  0000 C CNN
+F 1 "TEST_1P" V 2754 5172 50  0001 C CNN
+F 2 "wire_pads:SolderWirePad_single_1mmSMD" V 2741 5288 50  0001 L CNN
+F 3 "" H 2850 5100 50  0000 C CNN
+	1    2650 5100
 	0    -1   -1   0
 $EndComp
@@
 L devices:R_0603 R24
 U 1 1 5E341057
-P 5100 4900
-F 0 "R24" V 5050 4700 50  0000 C CNN
-F 1 "0R" V 5150 5050 50  0000 C CNN
-F 2 "resistors:R_0603" H 5100 4750 50  0001 C CNN
-F 3 "" H 5100 4900 50  0000 C CNN
-	1    5100 4900
+P 5100 4700
+F 0 "R24" V 5050 4500 50  0000 C CNN
+F 1 "0R" V 5150 4850 50  0000 C CNN
+F 2 "resistors:R_0603" H 5100 4550 50  0001 C CNN
+F 3 "" H 5100 4700 50  0000 C CNN
+	1    5100 4700
 	0    1    1    0
 $EndComp
@@
 L devices:R_0603 R23
 U 1 1 5E3420FD
-P 5100 4800
-F 0 "R23" V 5050 4600 50  0000 C CNN
-F 1 "0R" V 5150 4950 50  0000 C CNN
-F 2 "resistors:R_0603" H 5100 4650 50  0001 C CNN
-F 3 "" H 5100 4800 50  0000 C CNN
-	1    5100 4800
-	0    1    1    0
-$EndComp
-Wire Wire Line
-	5950 4900 5200 4900
-Wire Wire Line
-	5950 4800 5200 4800
-Wire Wire Line
-	3800 4800 5000 4800
-Wire Wire Line
-	3800 4900 5000 4900
-Text Label 5400 4800 0    50   ~ 0
+P 5100 4600
+F 0 "R23" V 5050 4400 50  0000 C CNN
+F 1 "0R" V 5150 4750 50  0000 C CNN
+F 2 "resistors:R_0603" H 5100 4450 50  0001 C CNN
+F 3 "" H 5100 4600 50  0000 C CNN
+	1    5100 4600
+	0    1    1    0
+$EndComp
+Wire Wire Line
+	5950 4700 5200 4700
+Wire Wire Line
+	5950 4600 5200 4600
+Wire Wire Line
+	3800 4600 5000 4600
+Wire Wire Line
+	3800 4700 5000 4700
+Text Label 5400 4600 0    50   ~ 0
 SDA
-Text Label 5400 4900 0    50   ~ 0
+Text Label 5400 4700 0    50   ~ 0
 SCL
 $Comp
@@
 LED_B
 Wire Wire Line
-	2450 5100 3300 5100
-Wire Wire Line
-	2450 5000 3300 5000
-Wire Wire Line
 	2450 4800 3300 4800
+Wire Wire Line
+	2450 4700 3300 4700
 $Comp
 L devices:LED_RGB D6
@@
 Wire Wire Line
 	5700 6450 5700 6500
+Wire Wire Line
+	3300 5000 2650 5000
+Wire Wire Line
+	4750 4500 3800 4500
+Text Notes 1200 5350 0    50   ~ 0
+Pin 1, 3, 5, 7, 17 and 19 \nare also connected to \nthe WiFi NINA module \non the Vidor 4000
 $EndSCHEMATC

Commit message: changed pinning to fit to https://github.com/107-systems/viper-vidor-fpga
Other:
- moved on the sheet: W9
Changed lines of the file:
@@
 Text Label 4200 5100 0    50   ~ 0
 VSYNC
-Text Label 2550 5300 0    50   ~ 0
+Text Label 2550 6500 0    50   ~ 0
 XCLK
 Text Label 4200 4800 0    50   ~ 0
@@
 Text Label 2550 6700 0    50   ~ 0
 DOUT9
-Text Label 2550 6500 0    50   ~ 0
+Text Label 2550 5800 0    50   ~ 0
 DOUT7
-Text Label 2550 5800 0    50   ~ 0
+Text Label 2550 5700 0    50   ~ 0
 DOUT5
 Text Label 4200 6500 0    50   ~ 0
@@
 Text Label 4200 5500 0    50   ~ 0
 HREF
-Text Label 2550 5400 0    50   ~ 0
+Text Label 2550 5300 0    50   ~ 0
 PCLK
 Text Label 4200 4900 0    50   ~ 0
@@
 Text Label 2550 6600 0    50   ~ 0
 DOUT8
-Text Label 2550 6400 0    50   ~ 0
+Text Label 2550 4800 0    50   ~ 0
 DOUT6
-Text Label 2550 5700 0    50   ~ 0
+Text Label 2550 5400 0    50   ~ 0
 DOUT4
 Text Label 4200 6400 0    50   ~ 0
@@
 Wire Wire Line
 	4500 5600 3800 5600
-Wire Wire Line
-	4500 4400 3800 4400
 Text Label 2750 4200 0    50   ~ 0
 RSVD0
@@
 Text Label 2750 4400 0    50   ~ 0
 RSVD2
-Text Label 4100 4400 0    50   ~ 0
+Text Label 2750 4700 0    50   ~ 0
 RSVD3
 Text Label 2750 4500 0    50   ~ 0
@@
 Text Label 4100 4700 0    50   ~ 0
 SCL_V
-Text Label 2550 4700 0    50   ~ 0
+Text Label 4100 4400 0    50   ~ 0
 LED_G
-Text Label 2550 4800 0    50   ~ 0
+Text Label 2550 6400 0    50   ~ 0
 LED_B
 $Comp
@@
 L mechanical-connectors:TEST_1P W9
 U 1 1 5E310C83
-P 4500 4400
-F 0 "W9" V 4454 4588 50  0000 L CNN
-F 1 "TEST_1P" V 4545 4588 50  0001 L CNN
-F 2 "wire_pads:SolderWirePad_single_1mmSMD" V 4591 4588 50  0001 L CNN
-F 3 "" H 4700 4400 50  0000 C CNN
-	1    4500 4400
-	0    1    1    0
+P 2650 4700
+F 0 "W9" V 2604 4888 50  0000 L CNN
+F 1 "TEST_1P" V 2695 4888 50  0001 L CNN
+F 2 "wire_pads:SolderWirePad_single_1mmSMD" V 2741 4888 50  0001 L CNN
+F 3 "" H 2850 4700 50  0000 C CNN
+	1    2650 4700
+	0    -1   -1   0
 $EndComp
 $Comp
@@
 Wire Wire Line
 	2450 4800 3300 4800
-Wire Wire Line
-	2450 4700 3300 4700
 $Comp
 L devices:LED_RGB D6
@@
 Text Notes 1200 5350 0    50   ~ 0
 Pin 1, 3, 5, 7, 17 and 19 \nare also connected to \nthe WiFi NINA module \non the Vidor 4000
+Wire Wire Line
+	3800 4400 4750 4400
+Wire Wire Line
+	3300 4700 2650 4700
 $EndSCHEMATC

Commit message: changed resistors for led from 1k to 3k3, added changes file
Parts:
- R25, R26, R27, R28, R29: value 1k -> 3k3
Changed lines of the file:
@@
 P 8000 6200
 F 0 "R29" V 7950 6000 50  0000 C CNN
-F 1 "1k" V 8050 6350 50  0000 C CNN
+F 1 "3k3" V 8050 6350 50  0000 C CNN
 F 2 "resistors:R_0603" H 8000 6050 50  0001 C CNN
 F 3 "" H 8000 6200 50  0000 C CNN
@@
 P 8000 5650
 F 0 "R28" V 7950 5450 50  0000 C CNN
-F 1 "1k" V 8050 5800 50  0000 C CNN
+F 1 "3k3" V 8050 5800 50  0000 C CNN
 F 2 "resistors:R_0603" H 8000 5500 50  0001 C CNN
 F 3 "" H 8000 5650 50  0000 C CNN
@@
 P 8000 5100
 F 0 "R27" V 7950 4900 50  0000 C CNN
-F 1 "1k" V 8050 5250 50  0000 C CNN
+F 1 "3k3" V 8050 5250 50  0000 C CNN
 F 2 "resistors:R_0603" H 8000 4950 50  0001 C CNN
 F 3 "" H 8000 5100 50  0000 C CNN
@@
 P 8000 4550
 F 0 "R26" V 7950 4350 50  0000 C CNN
-F 1 "1k" V 8050 4700 50  0000 C CNN
+F 1 "3k3" V 8050 4700 50  0000 C CNN
 F 2 "resistors:R_0603" H 8000 4400 50  0001 C CNN
 F 3 "" H 8000 4550 50  0000 C CNN
@@
 P 8000 4000
 F 0 "R25" V 7950 3800 50  0000 C CNN
-F 1 "1k" V 8050 4150 50  0000 C CNN
+F 1 "3k3" V 8050 4150 50  0000 C CNN
 F 2 "resistors:R_0603" H 8000 3850 50  0001 C CNN
 F 3 "" H 8000 4000 50  0000 C CNN

Commit message: updated symbold for vidor mpcie connector in schematic
Parts:
- removed CN1: TE_2041119-2, connectors_pci-express:MPCIe_4mm, symbol mechanical-connectors:CONN_02X26
- added CN1: TE_2041119-2, connectors_pci-express:MPCIe_4mm, symbol MODULE_compute:ARDUINO_VIDOR_MPCIE
Other:
- moved on the sheet: MECH1, MECH2, R23, R24, W1, W10, W2, W3, W4, W5, W9

Commit message: restored design files from master
Parts:
- removed CN1: TE_2041119-2, connectors_pci-express:MPCIe_4mm, symbol MODULE_compute:ARDUINO_VIDOR_MPCIE
- added CN1: TE_2041119-2, connectors_pci-express:MPCIe_4mm, symbol mechanical-connectors:CONN_02X26
Other:
- moved on the sheet: MECH1, MECH2, R23, R24, W1, W10, W2, W3, W4, W5, W9
